File: Electrical Design/KICAD_BTE_RIGID/Tympan_BTE_RIGID.kicad_pcb (KiCad board)
At the start: 2 copper layers, 5.3 x 6.8 mm, 5 parts, among them J1 Input Wire Connector, J2 FPC Connector, J3 CS44 Connector

Commit message: Labeled wire colors and swapped the +- speaker connections
Connections:
- J1 pad 5: /SPK+ -> /SPK-
- J1 pad 6: /SPK- -> /SPK+
- J3 pad 3: /SPK- -> /SPK+
- J3 pad 4: /SPK+ -> /SPK-
Routing:
- net /SPK-: track 3.27 -> 3.79 mm
- net /SPK+: track 3.79 -> 3.27 mm
Changed lines of the file:
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@@
     )
     (pad 4 smd rect (at -0.425 0 352.5) (size 0.5 1) (layers B.Cu B.Mask)
+      (net 6 /SPK-))
+    (pad 3 smd rect (at 0.425 0 352.5) (size 0.5 1) (layers B.Cu B.Mask)
       (net 1 /SPK+))
-    (pad 3 smd rect (at 0.425 0 352.5) (size 0.5 1) (layers B.Cu B.Mask)
-      (net 6 /SPK-))
     (pad 2 smd rect (at 0.425 0 352.5) (size 0.5 1) (layers F.Cu F.Mask)
       (net 8 "Net-(J3-Pad2)"))
@@
     )
     (pad 6 smd rect (at 0 1.75 90) (size 2 0.35) (layers F.Cu F.Mask)
+      (net 1 /SPK+))
+    (pad 5 smd rect (at 0 1.05 90) (size 2 0.35) (layers F.Cu F.Mask)
       (net 6 /SPK-))
-    (pad 5 smd rect (at 0 1.05 90) (size 2 0.35) (layers F.Cu F.Mask)
-      (net 1 /SPK+))
     (pad 4 smd rect (at 0 0.35 90) (size 2 0.35) (layers F.Cu F.Mask)
       (net 5 GND))
@@
   (gr_arc (start 123.978503 89.371938) (end 123.875305 89.758397) (angle -180) (layer Edge.Cuts) (width 0.05))
   (gr_arc (start 128.201259 89.927874) (end 128.124786 89.535252) (angle -180) (layer Edge.Cuts) (width 0.05))
-  (via (at 126.774187 90.271304) (size 0.4) (drill 0.1) (layers F.Cu B.Cu) (net 1))
-  (segment (start 126.974186 90.471303) (end 126.774187 90.271304) (width 0.1) (layer F.Cu) (net 1))
-  (segment (start 125.594183 89.221304) (end 125.514183 89.301304) (width 0.1) (layer B.Cu) (net 1))
-  (segment (start 127.074183 92.031304) (end 127.074183 90.5713) (width 0.1) (layer F.Cu) (net 1))
-  (segment (start 127.074183 90.5713) (end 126.974186 90.471303) (width 0.1) (layer F.Cu) (net 1))
-  (segment (start 125.514183 89.524156) (end 126.261331 90.271304) (width 0.1) (layer B.Cu) (net 1))
-  (segment (start 126.261331 90.271304) (end 126.491345 90.271304) (width 0.1) (layer B.Cu) (net 1))
-  (segment (start 125.514183 89.301304) (end 125.514183 89.524156) (width 0.1) (layer B.Cu) (net 1))
-  (segment (start 126.491345 90.271304) (end 126.774187 90.271304) (width 0.1) (layer B.Cu) (net 1))
+  (via (at 126.774187 90.271304) (size 0.4) (drill 0.1) (layers F.Cu B.Cu) (net 6))
+  (segment (start 126.974186 90.471303) (end 126.774187 90.271304) (width 0.1) (layer F.Cu) (net 6))
+  (segment (start 125.594183 89.221304) (end 125.514183 89.301304) (width 0.1) (layer B.Cu) (net 6))
+  (segment (start 127.074183 92.031304) (end 127.074183 90.5713) (width 0.1) (layer F.Cu) (net 6))
+  (segment (start 127.074183 90.5713) (end 126.974186 90.471303) (width 0.1) (layer F.Cu) (net 6))
+  (segment (start 125.514183 89.524156) (end 126.261331 90.271304) (width 0.1) (layer B.Cu) (net 6))
+  (segment (start 126.261331 90.271304) (end 126.491345 90.271304) (width 0.1) (layer B.Cu) (net 6))
+  (segment (start 125.514183 89.301304) (end 125.514183 89.524156) (width 0.1) (layer B.Cu) (net 6))
+  (segment (start 126.491345 90.271304) (end 126.774187 90.271304) (width 0.1) (layer B.Cu) (net 6))
   (via (at 124.274183 93.531314) (size 0.4) (drill 0.1) (layers F.Cu B.Cu) (net 2))
   (segment (start 124.274183 92.031304) (end 124.274183 93.531314) (width 0.1) (layer F.Cu) (net 2))
@@
   (via (at 127.744183 94.251304) (size 0.4) (drill 0.1) (layers F.Cu B.Cu) (net 5))
   (segment (start 126.839183 94.251304) (end 127.744183 94.251304) (width 0.1) (layer B.Cu) (net 5))
-  (segment (start 126.536082 89.331304) (end 127.22173 90.016952) (width 0.1) (layer B.Cu) (net 6))
-  (segment (start 127.621728 90.41695) (end 127.421729 90.216951) (width 0.1) (layer F.Cu) (net 6))
-  (via (at 127.421729 90.216951) (size 0.4) (drill 0.1) (layers F.Cu B.Cu) (net 6))
-  (segment (start 127.22173 90.016952) (end 127.421729 90.216951) (width 0.1) (layer B.Cu) (net 6))
-  (segment (start 127.774183 92.031304) (end 127.774183 90.569405) (width 0.1) (layer F.Cu) (net 6))
-  (segment (start 127.774183 90.569405) (end 127.621728 90.41695) (width 0.1) (layer F.Cu) (net 6))
-  (segment (start 126.474183 89.331304) (end 126.536082 89.331304) (width 0.1) (layer B.Cu) (net 6))
+  (segment (start 126.536082 89.331304) (end 127.22173 90.016952) (width 0.1) (layer B.Cu) (net 1))
+  (segment (start 127.621728 90.41695) (end 127.421729 90.216951) (width 0.1) (layer F.Cu) (net 1))
+  (via (at 127.421729 90.216951) (size 0.4) (drill 0.1) (layers F.Cu B.Cu) (net 1))
+  (segment (start 127.22173 90.016952) (end 127.421729 90.216951) (width 0.1) (layer B.Cu) (net 1))
+  (segment (start 127.774183 92.031304) (end 127.774183 90.569405) (width 0.1) (layer F.Cu) (net 1))
+  (segment (start 127.774183 90.569405) (end 127.621728 90.41695) (width 0.1) (layer F.Cu) (net 1))
+  (segment (start 126.474183 89.331304) (end 126.536082 89.331304) (width 0.1) (layer B.Cu) (net 1))
   (segment (start 127.744183 93.361304) (end 127.764183 93.341304) (width 0.1) (layer B.Cu) (net 9))
   (segment (start 126.494183 93.361304) (end 127.744183 93.361304) (width 0.1) (layer B.Cu) (net 9))
