File: Electrical Design/KICAD_BTE_RIGID/Tympan_BTE_RIGID_Array.kicad_pcb (KiCad board)
At the start: 2 copper layers, 49 x 21 mm, 25 parts, among them J1 Input Wire Connector, J2 FPC Connector, J3 CS44 Connector

Commit message: Labeled wire colors and swapped the +- speaker connections
Connections:
- C1 pad 1: (no net) -> +3V3 (x4)
- C1 pad 2: (no net) -> GND (x4)
- J1 pad 1: (no net) -> /DATA (x4)
- J1 pad 2: (no net) -> /CLK (x4)
- J1 pad 3: (no net) -> +3V3 (x4)
- J1 pad 4: (no net) -> GND (x4)
- J1 pad 5: (no net) -> /SPK- (x4)
- J1 pad 6: (no net) -> /SPK+ (x4)
- J1 pad 5: /SPK+ -> /SPK-
- J1 pad 6: /SPK- -> /SPK+
- J2 pad 1: (no net) -> GND (x4)
- J2 pad 2: (no net) -> /CLK (x4)
- J2 pad 3: (no net) -> +3V3 (x4)
- J2 pad 4: (no net) -> Net-(J2-Pad4) (x4)
- J2 pad 5: (no net) -> GND (x4)
- J2 pad 6: (no net) -> GND (x4)
- J3 pad 1: (no net) -> Net-(J3-Pad1) (x4)
- J3 pad 2: (no net) -> Net-(J3-Pad2) (x4)
- J3 pad 3: (no net) -> /SPK+ (x4)
- J3 pad 4: (no net) -> /SPK- (x4)
- J3 pad 3: /SPK- -> /SPK+
- J3 pad 4: /SPK+ -> /SPK-
- R1 pad 1: (no net) -> /DATA (x4)
- R1 pad 2: (no net) -> Net-(J2-Pad4) (x4)
Routing:
- net (no net): track 101.2 -> 0.00 mm, vias 28 -> 0
- net +3V3: track 5.49 -> 27.4 mm, vias 1 -> 5
- net /CLK: track 4.99 -> 24.9 mm, vias 1 -> 5
- net /SPK-: track 3.27 -> 18.9 mm, vias 1 -> 5
- net Net-(J2-Pad4): track 3.42 -> 17.1 mm
- net /SPK+: track 3.79 -> 16.4 mm, vias 1 -> 5
- net /DATA: track 2.68 -> 13.4 mm, vias 1 -> 5
- net GND: track 1.67 -> 8.33 mm, vias 2 -> 10
